File: minibaen r2.kicad_pcb (KiCad board)
At the start: 2 copper layers, 242.9 x 76.2 mm, 135 parts, among them SW1 SW_Push, SW2 RotaryEncoder_Switch, U1 ATmega32U2-A, U2 PRTR5V0U2X, Y1 Crystal_GND24_Small

Commit message: pub
Parts:
- MX14, MX40: footprint MX_Only:MXOnly-1U-NoLED -> MX_Only:MXOnly-1.25U-NoLED
- MX27: footprint MX_Only:MXOnly-1U-NoLED -> MX_Only:MXOnly-1.75U-NoLED

Commit message: add
Parts:
- removed the D21 at (171.2, 57.9)
- removed the D33 at (152.5, 77.0)
- removed the D44 at (121.2, 100.0)
- removed the D45 at (133.9, 96.0)
- removed the D47 at (170.9, 98.4)
- removed the D48 at (189.9, 96.0)
- removed H1, H2, H3: MountingHole, MountingHole:MountingHole_2.2mm_M2_DIN965_Pad
- removed the MX20 at (149.4, 57.1)
- removed the MX33 at (149.4, 76.2)
- removed the MX44 at (112.1, 95.2)
- removed the MX45 at (130.8, 95.2)
- removed the MX47 at (168.1, 95.2)
- removed MX53, MX57: MX-NoLED, MX_Only:MXOnly-2U-ReversedStabilizers-NoLED
- removed MX54, MX56, MX58: MX-NoLED, MX_Only:MXOnly-3U-ReversedStabilizers-NoLED
- removed MX55: MX-NoLED, MX_Only:MXOnly-7U-ReversedStabilizers-NoLED
- added D26: D_Small, Diode_SMD:D_SOD-123, B.Cu at (46.8, 86.2)
- added D43: D_Small, Diode_SMD:D_SOD-123, B.Cu at (157.2, 101.6)
- added MX26: MX-NoLED, MX_Only:MXOnly-1U-NoLED, F.Cu at (56.4, 81.8)
- added MX40: MX-NoLED, MX_Only:MXOnly-1U-NoLED, F.Cu at (208.8, 100.8)
- added MX41: MX-NoLED, MX_Only:MXOnly-1U-NoLED, F.Cu at (227.8, 100.8)
- added MX42: MX-NoLED, MX_Only:MXOnly-1U-NoLED, F.Cu at (246.9, 100.8)
- added MX43: MX-NoLED, MX_Only:MXOnly-1U-NoLED, F.Cu at (265.9, 100.8)
- MX25: renamed from MX26; footprint MX_Only:MXOnly-1U-NoLED -> MX_Only:MXOnly-1.5U-NoLED
- MX39: renamed from MX46; footprint MX_Only:MXOnly-1U-NoLED -> MX_Only:MXOnly-1.25U-NoLED
- MX46: renamed from MX42; footprint MX_Only:MXOnly-1U-NoLED -> MX_Only:MXOnly-1.25U-NoLED
- MX47: renamed from MX43; footprint MX_Only:MXOnly-1U-NoLED -> MX_Only:MXOnly-1.75U-NoLED
- MX48: footprint MX_Only:MXOnly-1U-NoLED -> MX_Only:MXOnly-2.25U-ReversedStabilizers-NoLED
- MX49: footprint MX_Only:MXOnly-1U-NoLED -> MX_Only:MXOnly-1.75U-NoLED
- MX50, MX52: footprint MX_Only:MXOnly-1U-NoLED -> MX_Only:MXOnly-1.25U-NoLED
- moved SW1 203.9 mm to (236.1, 72.2), turned to -90 degrees
- moved SW2 110.0 mm to (39.6, 81.5)
- moved MX39 38.3 mm to (187.3, 100.8)
- moved MX48 33.3 mm to (154.0, 100.8)
- moved D44 27.5 mm to (179.4, 101.6)
- moved D42 23.2 mm to (119.1, 101.6)
- moved MX47 23.2 mm to (115.9, 100.8)
- moved D32 21.6 mm to (154.8, 82.5)
- moved MX32 21.6 mm to (151.6, 81.8)
- moved D31 21.3 mm to (135.7, 82.5)
- moved MX31 21.2 mm to (132.6, 81.8)
- moved D30 20.9 mm to (116.7, 82.5)
- moved MX30 20.9 mm to (113.5, 81.8)
- moved D29 20.6 mm to (97.6, 82.5)
- moved MX29 20.5 mm to (94.5, 81.8)
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- renumbered C2 to C1, C4 to C2, C5 to C4, C6 to C5, C7 to C6, C1 to C7, D22 to D21, D23 to D22, D24 to D23, D25 to D24, D26 to D25, D34 to D33, D35 to D34, D36 to D35, D37 to D36, D38 to D37, D39 to D38, D40 to D39, D41 to D40, D42 to D41, D43 to D42, D46 to D44, D49 to D45, D50 to D46, D51 to D47, D52 to D48, MX21 to MX20, MX22 to MX21, MX23 to MX22, MX24 to MX23, MX25 to MX24, MX34 to MX33, MX35 to MX34, MX36 to MX35, MX37 to MX36, MX38 to MX37, MX39 to MX38, MX40 to MX44, MX41 to MX45
Connections:
- MX20 pad 2: Net-(D21-Pad2) (its old number) -> Net-(D20-Pad2)
- MX27 pad 1: col0 -> col1
- MX28 pad 1: col1 -> col2
- MX29 pad 1: col2 -> col3
- MX30 pad 1: col3 -> col4
- MX31 pad 1: col4 -> col5
- MX32 pad 1: col5 -> col6
- MX48 pad 1: col8 -> col5
- SW2 pad S2: col6 -> col0
Routing:
- net GND: track 48.5 -> 446.7 mm, vias 13 -> 21
- net Net-(R1-Pad2): track 221.9 -> 16.7 mm, vias 0 -> 2
- net encb: track 141.5 -> 303.5 mm, vias 5 -> 2
- net enca: track 151.7 -> 307.6 mm, vias 5 -> 2
- net row1: track 345.2 -> 222.8 mm, vias 7 -> 2
- net row0: track 348.4 -> 266.8 mm
- net col9: track 122.2 -> 171.5 mm, vias 2 -> 1
- net col12: track 120.3 -> 75.5 mm
- net col5: track 229.4 -> 197.2 mm, vias 2 -> 0
- net col10: track 116.2 -> 142.5 mm, vias 2 -> 1
- net col0: track 319.3 -> 294.8 mm, vias 1 -> 0
- net col8: track 163.2 -> 140.7 mm, vias 0 -> 3
- net col1: track 302.9 -> 283.7 mm, vias 1 -> 0
- net Net-(D45-Pad2): track 3.21 -> 21.2 mm
- net col4: track 228.3 -> 211.9 mm
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- removed copper zone on B.Cu, net GND
- removed copper zone on F.Cu, net GND

Commit message: add
Parts:
- C7: value 4.7n -> 4.7nF
- R5, R6: value 5k1 -> 5.1k
- SW1: footprint Connector_PinHeader_2.54mm:PinHeader_1x02_P2.54mm_Vertical -> Button_Switch_SMD:SW_Push_SPST_NO_Alps_SKRK
- U1: value ATmega32U2-A -> ATmega32U4-M; footprint Package_QFP:TQFP-32_7x7mm_P0.8mm -> Package_DFN_QFN:QFN-44-1EP_7x7mm_P0.5mm_EP5.2x5.2mm
- moved C3 10.3 mm to (237.3, 69.6)
- moved R4 8.07 mm to (257.1, 82.5), turned to 90 degrees
- moved D37 7.94 mm to (238.9, 84.9)
- moved D11 3.98 mm to (231.5, 48.4)
- moved D38 2.86 mm to (263.5, 86.5)
- moved R1 2.18 mm to (245.3, 73.8)
- moved SW1 1.59 mm to (236.1, 73.8)
- moved C5 1.57 mm to (253.2, 63.5)
- moved C6 1.56 mm to (268.3, 67.5)
- moved C4 0.98 mm to (250.3, 65.9)
- moved D13 0.80 mm to (269.1, 45.2)
- moved C7 0.54 mm to (252.6, 38.9)
- moved R7 0.54 mm to (238.5, 38.9)
- turned U1 to 135 degrees
Connections:
- U1 pad 10: col12 -> col10
- U1 pad 11: col10 -> col9
- U1 pad 12: col9 -> col8
- U1 pad 14: col8 -> col12
Routing:
- net GND: track 446.7 -> 60.9 mm, vias 21 -> 30
- net col8: track 140.7 -> 160.7 mm, vias 3 -> 5
- net +5V: track 91.0 -> 106.0 mm
- net Net-(C3-Pad1): track 4.93 -> 16.6 mm, vias 0 -> 2
- net col12: track 75.5 -> 85.9 mm, vias 2 -> 0
- net col9: track 171.5 -> 179.6 mm
- net col10: track 142.5 -> 150.3 mm
- net row3: track 265.9 -> 272.9 mm
- net encb: track 303.5 -> 310.0 mm
- net row0: track 266.8 -> 272.4 mm
- net enca: track 307.6 -> 312.3 mm
- net Net-(C1-Pad1): track 16.8 -> 21.1 mm
- net Net-(C2-Pad2): track 18.2 -> 22.3 mm
- net Net-(D11-Pad2): track 4.43 -> 8.48 mm
- net Net-(D38-Pad2): track 8.62 -> 12.6 mm
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- added copper zone on B.Cu, net GND
- added copper zone on F.Cu, net GND
