File: Plate/minibaen r2-plate.kicad_pcb (KiCad board)
At the start: 2 copper layers, 242.9 x 76.2 mm, 134 parts, among them SW1 SW_Push, SW2 RotaryEncoder_Switch, U1 ATmega32U2-A, U2 PRTR5V0U2X, Y1 Crystal_GND24_Small

Commit message: add
Parts:
- removed C1: 4.7n, rainfootprints:blank
- removed C2, C4: 22pF, rainfootprints:blank
- removed C3: 1uF, rainfootprints:blank
- removed C5, C6: 0.1uF, rainfootprints:blank
- removed C7: 10uF, rainfootprints:blank
- removed D1, D10, D11, D12, D13, D14, D15, D16, D17, D18, D19, D2, D20, D21, D22, D23, D24, D25, D26, D27, D28, D29, D3, D30, D31, D32, D33, D34, D35, D36, D37, D38, D39, D4, D40, D41, D42, D43, D44, D45, D46, D47, D48, D49, D5, D50, D51, D52, D6, D7, D8, D9: D_Small, rainfootprints:blank
- removed F1: 500mA, rainfootprints:blank
- removed H1, H2, H3: MountingHole, kbd:M2_Hole_TH_Outside
- removed MX1, MX10, MX11, MX12, MX13, MX14, MX15, MX16, MX17, MX18, MX19, MX2, MX20, MX21, MX22, MX23, MX24, MX25, MX26, MX27, MX28, MX29, MX3, MX30, MX31, MX32, MX33, MX34, MX35, MX36, MX37, MX38, MX39, MX4, MX5, MX6, MX7, MX8, MX9: MX-NoLED, rainfootprints:1u-cutout
- removed MX41, MX42, MX43, MX44, MX45, MX46, MX47, MX48, MX49, MX50, MX51, MX52, MX53, MX54, MX55, MX56, MX57, MX58: MX-NoLED, rainfootprints:blank
- removed R1, R4: 10k, rainfootprints:blank
- removed R2, R3: 22, rainfootprints:blank
- removed R5, R6: 5k1, rainfootprints:blank
- removed R7: 1M, rainfootprints:blank
- removed SW1: SW_Push, rainfootprints:blank
- removed SW2: RotaryEncoder_Switch, rainfootprints:blank
- removed U1: ATmega32U2-A, rainfootprints:blank
- removed U2: PRTR5V0U2X, rainfootprints:blank
- removed USB1: HRO-TYPE-C-31-M-12, rainfootprints:blank
- removed Y1: Crystal_GND24_Small, rainfootprints:blank
Routing:
- removed copper zone on B.Cu, net (none)
- removed copper zone on F.Cu, net (none)
Other:
- board size 242.9 x 76.2 mm -> 241.8 x 85.1 mm
- board text added: "concept by Taylor r2 pcb by rain v1.0"
